Commit message: update planar gps imu back_camara

File: wamv_gazebo/urdf/components/wamv_gps.xacro (robot description, xacro)
@@ -28,5 +28,5 @@
       </inertial>
     </link>
-    <joint name="${namespace}/${name}_joint" type="revolute">
+    <joint name="${namespace}/${name}_joint" type="fixed">
       <axis xyz="0 0 1"/>
       <limit effort="1000.0" lower="0.0" upper="0" velocity="0"/>

File: wamv_gazebo/urdf/components/wamv_planar_lidar.xacro (robot description, xacro)
@@ -19,5 +19,7 @@
     <gazebo reference="${namespace}/${name}_link">
       <sensor type="gpu_ray" name="multibeam_sensor_${name}">
+      <always_on>true</always_on>
         <update_rate>10</update_rate>
+        <visualize>true</visualize>
         <ray>
           <scan>

File: wamv_gazebo/urdf/wamv_gazebo.urdf.xacro (robot description, xacro)
@@ -73,5 +73,5 @@
   <xacro:if value="$(arg camera_enabled)">
       <xacro:wamv_camera name="front_camera" y="0" x="1.6" z="0.65" />
-      <xacro:wamv_camera name="back_camera" y="0" x="0.30" z="0.65" P="${radians(-180)}"/>
+      <xacro:wamv_camera name="back_camera" y="0" x="0.30" z="0.65" P="${radians(-180)}" R="${radians(-180)}"/>
   </xacro:if>
   <!--  GPS -->
@@ -89,5 +89,5 @@
   <!--  PLANAR -->
   <xacro:if value="$(arg planar_enabled)">
-    <xacro:wamv_multibeam_laser name="planar_wamv" x="0.6" y="0" z="0.65"/>
+    <xacro:wamv_multibeam_laser name="planar_wamv" x="0.6" y="0" z="0.7"/>
   </xacro:if>
 </robot>
