Commit message: centro de masa

File: wamv_description/urdf/thrusters/engine.xacro (robot description, xacro)
@@ -12,5 +12,5 @@
        -->
       <collision name="${prefix}_engine_vertical_axis_collision">
-        <origin xyz="-0.16 0 -0.24" rpy="0 0 0" />
+        <origin xyz="-0.16 0 -0.24" rpy="0 0 0" /> <!-- xyz="-0.16 0 -0.24" -->
         <geometry>
           <box size="0.2 0.15 0.83" />
@@ -18,5 +18,5 @@
       </collision>
       <collision name="${prefix}_engine_rear_end_collision">
-        <origin xyz="-0.34 0 0.12" rpy="0 0 0" />
+        <origin xyz="-0.34 0 0.12" rpy="0 0 0" /> <!-- xyz="-0.34 0 0.12" -->
         <geometry>
           <box size="0.12 0.15 0.12" />
@@ -35,5 +35,5 @@
       </visual>
       <collision name="${prefix}_propeller_collision">
-        <origin xyz="0 0 0" rpy="0 1.57 0" />
+        <origin xyz="0 0 0" rpy="0 1.57 0" /> <!-- xyz="0 0 0" -->
         <geometry>
           <cylinder length="0.18" radius="0.24" />
@@ -48,13 +48,13 @@
       <axis xyz="0 0 1"/>
       <limit lower="${-pi}" upper="${pi}" effort="10" velocity="10"/>
-      <origin xyz="${position}" rpy="${orientation}"/>
+      <origin xyz="${position}" rpy="${orientation}"/> <!-- xyz="${position}"-->
       <parent link="${namespace}/base_link"/>
       <child link="${namespace}/${prefix}_engine_link"/>
     </joint>
     <joint name="${namespace}/${prefix}_engine_propeller_joint" type="continuous">
-      <axis rpy="0 0 0" xyz="1 0 0"/>
+      <axis rpy="0 0 0" xyz="1 0 0"/>  <!-- xyz="1 0 0" -->
       <parent link="${namespace}/${prefix}_engine_link"/>
       <child link="${namespace}/${prefix}_propeller_link"/>
-      <origin rpy="0 0 0" xyz="-0.278156 0 -0.509371"/>
+      <origin rpy="0 0 0" xyz="-0.278156 0 -0.509371"/> <!-- xyz="-0.278156 0 -0.509371" -->
       <limit effort="100" velocity="100" />
       <dynamics friction="0.05" damping="0.05" />

File: wamv_description/urdf/wamv_base.urdf.xacro (robot description, xacro)
@@ -7,5 +7,5 @@
 <!-- Top part -->
     <collision name="topPart">
-      <origin xyz="0.95 0.0 0.5"/>
+      <origin xyz="0.95 0.0 0.5"/> <!-- xyz="0.95 0.0 0.5"-->
       <geometry>
         <box size="1.5 1.1 0.12"/>
@@ -14,5 +14,5 @@
     <!-- External sides -->
     <collision name="${prefix}_externalSide">
-      <origin xyz="${0.95-0.05} ${((0.5-0.06875)*reflect)} ${0.5-0.29}"/>
+      <origin xyz="${0.95-0.05} ${((0.5-0.06875)*reflect)} ${0.5-0.29}"/> <!-- xyz="${0.95-0.05} ${((0.5-0.06875)*reflect)} ${0.5-0.29}" -->
       <geometry>
         <box size="1.35 0.13 0.67"/>
@@ -21,5 +21,5 @@
     <!-- Internal sides -->
     <collision name="$prefix_internalSide">
-      <origin xyz="${0.95-0.05} ${((0.446875-0.06875-0.065)*reflect)} ${0.5-0.25}"/>
+      <origin xyz="${0.95-0.05} ${((0.446875-0.06875-0.065)*reflect)} ${0.5-0.25}"/> <!-- xyz="${0.95-0.05} ${((0.446875-0.06875-0.065)*reflect)} ${0.5-0.25}" -->
       <geometry>
         <box size="1.35 0.15625 0.5"/>
@@ -28,5 +28,5 @@
    <!-- Center part -->
     <collision name="centerPart">
-      <origin xyz="${0.95-0.6125} 0.0 ${0.5-0.25}"/>
+      <origin xyz="${0.95-0.6125} 0.0 ${0.5-0.25}"/> <!-- xyz="${0.95-0.6125} 0.0 ${0.5-0.25}"-->
       <geometry>
         <box size="0.20 0.5 0.5"/>
@@ -35,5 +35,5 @@
    <!-- Botoom part -->
     <collision name="bottomPart">
-      <origin xyz="0.95 0.0 ${0.5-0.25-0.365}"/>
+      <origin xyz="0.95 0.0 ${0.5-0.25-0.365}"/> <!-- xyz="0.95 0.0 ${0.5-0.25-0.365}" -->
       <geometry>
         <box size="1.3 0.55 0.285"/>
@@ -128,5 +128,5 @@
   <link name="${namespace}/dummy_link">
     <visual>
-      <origin xyz="0 0.085 -0.45" rpy="0 0 0" />
+      <origin xyz="-0.7 0.085 -0.45" rpy="0 0 0" />
       <geometry>
         <mesh filename="package://wamv_description/models/WAM-V-Base/mesh/WAM-V-Base.dae"/>

File: wamv_gazebo/urdf/thruster_layouts/wamv_t_thrusters.xacro (robot description, xacro)
@@ -2,8 +2,8 @@
 <robot xmlns:xacro="http://ros.org/wiki/xacro">
   <xacro:include filename="$(find wamv_description)/urdf/thrusters/engine.xacro" />
-  <xacro:engine prefix="left" position="${0.95+0.38} ${0.33} 0.368237" orientation="0.0 0.0 0.0" />
-  <xacro:engine prefix="right" position="${0.95+0.38} ${-0.33} 0.368237"  orientation="0.0 0.0 0.0" />
-  <xacro:engine prefix="middle" position="${0.68} ${0} 0.265237" orientation="0.0 0.0 0.0"/>
-  <xacro:engine prefix="lateral" position="${0.75} ${-0.25} 0.3" orientation="0.0 0.0 80.0"/>
+  <xacro:engine prefix="left" position="${0.95+0.38-0.7} ${0.33} 0.368237" orientation="0.0 0.0 0.0" />
+  <xacro:engine prefix="right" position="${0.95+0.38-0.7} ${-0.33} 0.368237"  orientation="0.0 0.0 0.0" />
+  <xacro:engine prefix="middle" position="${0.68-0.7} ${0} 0.265237" orientation="0.0 0.0 0.0"/>
+  <xacro:engine prefix="lateral" position="${0.75-0.7} ${-0.25} 0.3" orientation="0.0 0.0 80.0"/>
   <gazebo>
     <plugin name="wamv_gazebo_thrust" filename="libusv_gazebo_thrust_plugin.so">

File: wamv_gazebo/urdf/wamv_gazebo.urdf.xacro (robot description, xacro)
@@ -61,33 +61,33 @@
   <!-- === Sonar === -->
   <xacro:if value="$(arg sonar_enabled)">
-	<xacro:sonar name="sonar_sensor5" x="1.6" y="0.4" z="0.6" ros_topic="sonar5/distance5" Y="${radians(45)}" update_rate="10" min_range="0.3" max_range="2" field_of_view="56" ray_count="2" />
-	<xacro:sonar name="sonar_sensor4" x="1.6" y="0" z="0.6" ros_topic="sonar4/distance4" Y="${radians(0)}" update_rate="10" min_range="0.3" max_range="2" field_of_view="56" ray_count="2" />
-    	<xacro:sonar name="sonar_sensor3" x="1.6" y="-0.4" z="0.6" ros_topic="sonar3/distance3" Y="${radians(-45)}" update_rate="10" min_range="0.3" max_range="2" field_of_view="56" ray_count="2" />
-	<xacro:sonar name="sonar_sensor2" x="0.9" y="-0.4" z="0.6" ros_topic="sonar2/distance2" Y="${radians(-90)}" update_rate="10" min_range="0.3" max_range="2" field_of_view="56" ray_count="2" />
-    	<xacro:sonar name="sonar_sensor1" x="0.3" y="0.4" z="0.6" ros_topic="sonar1/distance1" Y="${radians(135)}" update_rate="10" min_range="0.3" max_range="2" field_of_view="56" ray_count="2" />
-	<xacro:sonar name="sonar_sensor8" x="0.3" y="0" z="0.6" ros_topic="sonar8/distance8" Y="${radians(180)}" update_rate="10" min_range="0.3" max_range="2" field_of_view="56" ray_count="2" />
-    	<xacro:sonar name="sonar_sensor7" x="0.3" y="-0.4" z="0.6" ros_topic="sonar7/distance7" Y="${radians(-135)}" update_rate="10" min_range="0.3" max_range="2" field_of_view="56" ray_count="2" />
-	<xacro:sonar name="sonar_sensor6" x="0.9" y="0.4" z="0.6" ros_topic="sonar6/distance6" Y="${radians(90)}" update_rate="10" min_range="0.3" max_range="2" field_of_view="56" ray_count="2" />
+	<xacro:sonar name="sonar_sensor5" x="0.9" y="0.4" z="0.6" ros_topic="sonar5/distance5" Y="${radians(45)}" update_rate="10" min_range="0.3" max_range="2" field_of_view="56" ray_count="2" />
+	<xacro:sonar name="sonar_sensor4" x="0.9" y="0" z="0.6" ros_topic="sonar4/distance4" Y="${radians(0)}" update_rate="10" min_range="0.3" max_range="2" field_of_view="56" ray_count="2" />
+    	<xacro:sonar name="sonar_sensor3" x="0.9" y="-0.4" z="0.6" ros_topic="sonar3/distance3" Y="${radians(-45)}" update_rate="10" min_range="0.3" max_range="2" field_of_view="56" ray_count="2" />
+	<xacro:sonar name="sonar_sensor2" x="0.2" y="-0.4" z="0.6" ros_topic="sonar2/distance2" Y="${radians(-90)}" update_rate="10" min_range="0.3" max_range="2" field_of_view="56" ray_count="2" />
+    	<xacro:sonar name="sonar_sensor1" x="-0.4" y="0.4" z="0.6" ros_topic="sonar1/distance1" Y="${radians(135)}" update_rate="10" min_range="0.3" max_range="2" field_of_view="56" ray_count="2" />
+	<xacro:sonar name="sonar_sensor8" x="-0.4" y="0" z="0.6" ros_topic="sonar8/distance8" Y="${radians(180)}" update_rate="10" min_range="0.3" max_range="2" field_of_view="56" ray_count="2" />
+    	<xacro:sonar name="sonar_sensor7" x="-0.4" y="-0.4" z="0.6" ros_topic="sonar7/distance7" Y="${radians(-135)}" update_rate="10" min_range="0.3" max_range="2" field_of_view="56" ray_count="2" />
+	<xacro:sonar name="sonar_sensor6" x="0.2" y="0.4" z="0.6" ros_topic="sonar6/distance6" Y="${radians(90)}" update_rate="10" min_range="0.3" max_range="2" field_of_view="56" ray_count="2" />
   </xacro:if>
   <!-- Cameras -->
   <xacro:if value="$(arg camera_enabled)">
-      <xacro:wamv_camera name="front_camera" y="0" x="1.6" z="0.65" />
-      <xacro:wamv_camera name="back_camera" y="0" x="0.30" z="0.65" P="${radians(-180)}" R="${radians(-180)}"/>
+      <xacro:wamv_camera name="front_camera" y="0" x="0.9" z="0.65" />
+      <xacro:wamv_camera name="back_camera" y="0" x="-0.4" z="0.65" P="${radians(-180)}" R="${radians(-180)}"/>
   </xacro:if>
   <!--  GPS -->
   <xacro:if value="$(arg gps_enabled)">
-    <xacro:wamv_gps name="gps_wamv" x="0.65" y="0" z="0.3" />
+    <xacro:wamv_gps name="gps_wamv" x="0" y="0" z="0.3" />
   </xacro:if>
   <!--  IMU -->
   <xacro:if value="$(arg imu_enabled)">
-    <xacro:wamv_imu name="imu_wamv" x="1.2" y="0" z="0.3" />
+    <xacro:wamv_imu name="imu_wamv" x="0.5" y="0" z="0.3" />
   </xacro:if>
   <!--  3D LIDAR -->
   <xacro:if value="$(arg lidar_enabled)">
-    <xacro:lidar name="lidar_wamv" x="0.6" y="0" z="0.65" type="16_beam"/>
+    <xacro:lidar name="lidar_wamv" x="-0.1" y="0" z="0.65" type="16_beam"/>
   </xacro:if>
   <!--  PLANAR -->
   <xacro:if value="$(arg planar_enabled)">
-    <xacro:wamv_multibeam_laser name="planar_wamv" x="0.6" y="0" z="0.8"/>
+    <xacro:wamv_multibeam_laser name="planar_wamv" x="-0.1" y="0" z="0.8"/>
   </xacro:if>
 </robot>
