Commit message: agregado arbol trasnformadas
modificacion para que tome arbol de transformadas propio

File: wamv_description/urdf/wamv_base.urdf.xacro (robot description, xacro)
@@ -5,117 +5,4 @@
   <!-- Macro for creating the main collisions as simple shapes. -->
   <xacro:macro name="main_collisions" params="prefix reflect:=1">
-<!-- Top part -->
-    <collision name="topPart">
-      <origin xyz="0.95 0.0 0.5"/> <!-- xyz="0.95 0.0 0.5"-->
-      <geometry>
-        <box size="1.5 1.1 0.12"/>
-      </geometry>
-    </collision>
-    <!-- External sides -->
-    <collision name="${prefix}_externalSide">
-      <origin xyz="${0.95-0.05} ${((0.5-0.06875)*reflect)} ${0.5-0.29}"/> <!-- xyz="${0.95-0.05} ${((0.5-0.06875)*reflect)} ${0.5-0.29}" -->
-      <geometry>
-        <box size="1.35 0.13 0.67"/>
-      </geometry>
-    </collision>
-    <!-- Internal sides -->
-    <collision name="$prefix_internalSide">
-      <origin xyz="${0.95-0.05} ${((0.446875-0.06875-0.065)*reflect)} ${0.5-0.25}"/> <!-- xyz="${0.95-0.05} ${((0.446875-0.06875-0.065)*reflect)} ${0.5-0.25}" -->
-      <geometry>
-        <box size="1.35 0.15625 0.5"/>
-      </geometry>
-    </collision>
-   <!-- Center part -->
-    <collision name="centerPart">
-      <origin xyz="${0.95-0.6125} 0.0 ${0.5-0.25}"/> <!-- xyz="${0.95-0.6125} 0.0 ${0.5-0.25}"-->
-      <geometry>
-        <box size="0.20 0.5 0.5"/>
-      </geometry>
-    </collision>
-   <!-- Botoom part -->
-    <collision name="bottomPart">
-      <origin xyz="0.95 0.0 ${0.5-0.25-0.365}"/> <!-- xyz="0.95 0.0 ${0.5-0.25-0.365}" -->
-      <geometry>
-        <box size="1.3 0.55 0.285"/>
-      </geometry>
-    </collision>
-    <!-- Main float
-    <collision name="${prefix}_float">
-      <origin xyz="-0.4 ${1.03*reflect} 0.2" rpy="${0*reflect} 1.57 0" />
-      <geometry>
-        <cylinder length="4" radius="0.2" />
-      </geometry>
-    </collision>
-    <collision name="${prefix}_mid_float">
-      <origin xyz="1.85 ${1.03*reflect} 0.3" rpy="${0*reflect} 1.38 0" />
-      <geometry>
-        <cylinder length="0.5" radius="0.17" />
-      </geometry>
-    </collision>
-    <collision name="${prefix}_front_float">
-      <origin xyz="2.3 ${1.03*reflect} 0.4" rpy="${0*reflect} 1.3 0" />
-      <geometry>
-        <cylinder length="0.45" radius="0.12" />
-      </geometry>
-    </collision>
-     Front beam
-    <collision name="front_${prefix}_beam_lower">
-      <origin xyz="0.9 ${0.85*reflect} 1" rpy="${0.78*reflect} 0 0" />
-      <geometry>
-        <cylinder length="0.5" radius="0.04" />
-      </geometry>
-    </collision>
-    <collision name="front_${prefix}_beam_upper">
-      <origin xyz="0.9 ${0.6*reflect} 1.18" rpy="${1.35*reflect} 0 0" />
-      <geometry>
-        <cylinder length="0.2" radius="0.04" />
-      </geometry>
-    </collision>
-     Mid beam
-    <collision name="mid_${prefix}_beam_lower">
-      <origin xyz="-0.65 ${0.99*reflect} 0.7" rpy="${0.1*reflect} 0.25 0" />
-      <geometry>
-        <cylinder length="0.45" radius="0.03" />
-      </geometry>
-    </collision>
-    <collision name="mid_${prefix}_beam_medium">
-      <origin xyz="-0.57 ${0.87*reflect} 1.05" rpy="${0.75*reflect} 0.25 0" />
-      <geometry>
-        <cylinder length="0.32" radius="0.03" />
-      </geometry>
-    </collision>
-    <collision name="mid_${prefix}_beam_upper">
-      <origin xyz="-0.55 ${0.65*reflect} 1.17" rpy="${1.35*reflect} 0.25 0" />
-      <geometry>
-        <cylinder length="0.3" radius="0.03" />
-      </geometry>
-    </collision>
-     Rear beam
-    <collision name="rear_${prefix}_beam_lower">
-      <origin xyz="-0.74 ${1.03*reflect} 0.7" rpy="${0*reflect} -0.15 0" />
-      <geometry>
-        <cylinder length="0.45" radius="0.03" />
-      </geometry>
-    </collision>
-    <collision name="rear_${prefix}_beam_medium">
-      <origin xyz="-0.79 ${0.91*reflect} 1.05" rpy="${0.75*reflect} -0.15 0" />
-      <geometry>
-        <cylinder length="0.32" radius="0.03" />
-      </geometry>
-    </collision>
-    <collision name="rear_${prefix}_beam_upper">
-      <origin xyz="-0.81 ${0.67*reflect} 1.18" rpy="${1.45*reflect} -0.15 0" />
-      <geometry>
-        <cylinder length="0.3" radius="0.03" />
-      </geometry>
-    </collision>
--->
-    <!-- Joint
-    <collision name="${prefix}_joint">
-      <origin xyz="0.58 ${1.03*reflect} 0.6" rpy="${0*reflect} -0.6 0" />
-      <geometry>
-        <box size="0.65 0.2 0.1" />
-      </geometry>
-    </collision>-->
   </xacro:macro>
   <link name="${namespace}/base_link">
@@ -133,17 +20,13 @@
       </geometry>
     </visual>
-    <!-- Left base collisions -->
-    <xacro:main_collisions prefix="left" reflect="1" />
-    <!-- Right side collisions -->
-    <xacro:main_collisions prefix="right" reflect="-1" />
-     <!-- Top base -->
+     <!-- General collison for all robot made by JL -->
     <collision name="top_base">
-      <origin xyz="0 -0 1.25" rpy="0 0 0" />
+      <origin xyz="0.25 0  0.2" rpy="0 0 0" />
       <geometry>
-        <box size="1.85 1 0.1" />
+        <box size="1.52 1.16 .8" />
       </geometry>
     </collision>
     <inertial>
-      <!-- From WAM-V spec sheet -->
+      <!-- valore aproximados para Geneseas, chequear -->
       <mass value="16.32"/>
       <inertia ixx="2.74" ixy="0.0" ixz="0.0" iyy="4.16" iyz="0.0" izz="4.7"/>

File: wamv_gazebo/urdf/components/sonar_sensor.xacro (robot description, xacro)
@@ -67,5 +67,5 @@
           <gaussianNoise>0.005</gaussianNoise>
           <topicName>${ros_topic}</topicName>
-          <frameId>${namespace}/${name}_link</frameId>
+          <frameId>geneseas/${name}_link</frameId>
         </plugin>
       </sensor>

File: wamv_gazebo/urdf/components/wamv_camera.xacro (robot description, xacro)
@@ -157,8 +157,8 @@
           <alwaysOn>true</alwaysOn>
           <updateRate>0.0</updateRate>
-          <cameraName>${namespace}/${sensor_namespace}${camera_namespace}${name}</cameraName>
+          <cameraName>geneseas/${camera_namespace}${name}</cameraName>
           <imageTopicName>image_raw</imageTopicName>
           <cameraInfoTopicName>camera_info</cameraInfoTopicName>
-          <frameName>${namespace}/${name}_link_optical</frameName>
+          <frameName>geneseas/${name}_link</frameName>
           <hackBaseline>0.07</hackBaseline>
           <distortionK1>0.0</distortionK1>

File: wamv_gazebo/urdf/components/wamv_gps_original.xacro (robot description, xacro)
@@ -41,6 +41,6 @@
         <bodyName>${namespace}/${name}_link</bodyName>
         <!-- Manually prepend namespace to tf frame. -->
-        <frameId>geneseas/gps_link</frameId>
-       <topicName>/geneseas/gps/fix</topicName>
+        <frameId>${namespace}/${name}_link</frameId>
+        <topicName>${namespace}/${sensor_namespace}gps/gps/fix</topicName>
         <!-- Note that the hector_gazebo_ros_gps plugin uses NWU coordinates
              for reporting velocities.  This may cause problems if localization

File: wamv_gazebo/urdf/components/wamv_imu_original.xacro (robot description, xacro)
@@ -27,8 +27,8 @@
         <updateRate>${update_rate}</updateRate>
         <bodyName>${namespace}/${name}_link</bodyName>
-	<topicName>/geneseas/imu/data</topicName>
+        <topicName>${namespace}/${sensor_namespace}imu/imu/data</topicName>
         <serviceName>${namespace}/${sensor_namespace}imu_service</serviceName>
         <!-- Manually prepend namespace to tf frame. -->
-        <frameId>geneseas/imu_link</frameId>
+        <frameId>${namespace}/${name}_link</frameId>
         <alwaysOn>true</alwaysOn>
         <accelOffset>0.0 0.0 0.0</accelOffset>

File: wamv_gazebo/urdf/components/wamv_planar_lidar.xacro (robot description, xacro)
@@ -41,6 +41,6 @@
         </ray>
         <plugin name="multibeam_simulator" filename="libgazebo_ros_laser.so">
-          <topicName>${namespace}/${sensor_namespace}lidars/${name}/scan</topicName>
-          <frameName>${namespace}/${name}_link</frameName>
+          <topicName>/geneseas/lidar/planar/scan</topicName>
+          <frameName>geneseas/lidar_link</frameName>
         </plugin>
       </sensor>

File: wamv_gazebo/urdf/wamv_gazebo.urdf.xacro (robot description, xacro)
@@ -61,12 +61,12 @@
   <!-- === Sonar === -->
   <xacro:if value="$(arg sonar_enabled)">
-	<xacro:sonar name="sonar_sensor5" x="0.9" y="0.4" z="0.6" ros_topic="sonar5/distance5" Y="${radians(45)}" update_rate="10" min_range="0.3" max_range="2" field_of_view="56" ray_count="2" />
-	<xacro:sonar name="sonar_sensor4" x="0.9" y="0" z="0.6" ros_topic="sonar4/distance4" Y="${radians(0)}" update_rate="10" min_range="0.3" max_range="2" field_of_view="56" ray_count="2" />
-    	<xacro:sonar name="sonar_sensor3" x="0.9" y="-0.4" z="0.6" ros_topic="sonar3/distance3" Y="${radians(-45)}" update_rate="10" min_range="0.3" max_range="2" field_of_view="56" ray_count="2" />
-	<xacro:sonar name="sonar_sensor2" x="0.2" y="-0.4" z="0.6" ros_topic="sonar2/distance2" Y="${radians(-90)}" update_rate="10" min_range="0.3" max_range="2" field_of_view="56" ray_count="2" />
-    	<xacro:sonar name="sonar_sensor1" x="-0.4" y="0.4" z="0.6" ros_topic="sonar1/distance1" Y="${radians(135)}" update_rate="10" min_range="0.3" max_range="2" field_of_view="56" ray_count="2" />
-	<xacro:sonar name="sonar_sensor8" x="-0.4" y="0" z="0.6" ros_topic="sonar8/distance8" Y="${radians(180)}" update_rate="10" min_range="0.3" max_range="2" field_of_view="56" ray_count="2" />
-    	<xacro:sonar name="sonar_sensor7" x="-0.4" y="-0.4" z="0.6" ros_topic="sonar7/distance7" Y="${radians(-135)}" update_rate="10" min_range="0.3" max_range="2" field_of_view="56" ray_count="2" />
-	<xacro:sonar name="sonar_sensor6" x="0.2" y="0.4" z="0.6" ros_topic="sonar6/distance6" Y="${radians(90)}" update_rate="10" min_range="0.3" max_range="2" field_of_view="56" ray_count="2" />
+	<xacro:sonar name="sonar_sensor5" x="0.9" y="0.4" z="0.6" ros_topic="/geneseas/sonar5/distance" Y="${radians(45)}" update_rate="10" min_range="0.3" max_range="2" field_of_view="56" ray_count="2" />
+	<xacro:sonar name="sonar_sensor4" x="0.9" y="0" z="0.6" ros_topic="/geneseas/sonar4/distance" Y="${radians(0)}" update_rate="10" min_range="0.3" max_range="2" field_of_view="56" ray_count="2" />
+ 	<xacro:sonar name="sonar_sensor3" x="0.9" y="-0.4" z="0.6" ros_topic="/geneseas/sonar3/distance" Y="${radians(-45)}" update_rate="10" min_range="0.3" max_range="2" field_of_view="56" ray_count="2" />
+	<xacro:sonar name="sonar_sensor2" x="0.2" y="-0.4" z="0.6" ros_topic="/geneseas/sonar2/distance" Y="${radians(-90)}" update_rate="10" min_range="0.3" max_range="2" field_of_view="56" ray_count="2" />
+ 	<xacro:sonar name="sonar_sensor1" x="-0.4" y="0.4" z="0.6" ros_topic="/geneseas/sonar1/distance" Y="${radians(135)}" update_rate="10" min_range="0.3" max_range="2" field_of_view="56" ray_count="2" />
+	<xacro:sonar name="sonar_sensor8" x="-0.4" y="0" z="0.6" ros_topic="/geneseas/sonar8/distance" Y="${radians(180)}" update_rate="10" min_range="0.3" max_range="2" field_of_view="56" ray_count="2" />
+ 	<xacro:sonar name="sonar_sensor7" x="-0.4" y="-0.4" z="0.6" ros_topic="/geneseas/sonar7/distance" Y="${radians(-135)}" update_rate="10" min_range="0.3" max_range="2" field_of_view="56" ray_count="2" />
+	<xacro:sonar name="sonar_sensor6" x="0.2" y="0.4" z="0.6" ros_topic="/geneseas/sonar6/distance" Y="${radians(90)}" update_rate="10" min_range="0.3" max_range="2" field_of_view="56" ray_count="2" />
   </xacro:if>
   <!-- Cameras -->
